File: appleii.vga.kicad_sch (KiCad schematic)
At the start: 32 parts, among them J1 BUS_APPLE_II, J2 Conn_01x25, J3 Conn_01x25, J4 Conn_01x08, J5 Conn_01x03, Q1 DMG2305UX, U1 74LVC245A, U2 74LVC245A, U3 74LVC245A, U4 74LVC245A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

Commit message: update board to v1.1.0
Some minor improvements based on v1.0.2 fab, assembly and test:
- correct "1uF" to "0.1uF" on decoupling caps
- reduce width of card edge connector by ~1.2mm
- increase trace widths to VCC and GND pins
- increase ground fill edge exclusion from 0 to 0.625mm
Parts:
- C1, C2, C3, C4: value 1uF -> 0.1uF
Other:
- note added: "v1.1.0 Changes: - correct "1uF" to "0.1uF" on decoupling caps - reduce width of card edge connector by ~1.2mm - increase trace widths to VCC and GND pins - increase ground fill edge exclusion from 0 to 0.625mm"
Changed lines of the file:
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@@
   (title_block
     (title "Apple II VGA")
-    (date "2023-07-05")
-    (rev "V1.0.2")
+    (date "2023-07-13")
+    (rev "v1.1.0")
     (company "swetland@frotz.net")
   )
@@
     (stroke (width 0) (type default))
   )
+  (text "v1.1.0 Changes:\n- correct \"1uF\" to \"0.1uF\" on decoupling caps\n- reduce width of card edge connector by ~1.2mm\n- increase trace widths to VCC and GND pins\n- increase ground fill edge exclusion from 0 to 0.625mm"
+    (at 160.02 168.91 0)
+    (effects (font (size 1.27 1.27)) (justify left bottom))
+  )
   (label "CLK_3.68M" (at 77.47 71.12 0) (fields_autoplaced)
     (effects (font (size 1.27 1.27)) (justify left bottom))
@@
       (effects (font (size 1.27 1.27)))
     )
-    (property "Value" "1uF" (at 195.58 128.27 90)
+    (property "Value" "0.1uF" (at 195.58 128.27 90)
       (effects (font (size 1.27 1.27)))
     )
@@
       (effects (font (size 1.27 1.27)))
     )
-    (property "Value" "1uF" (at 195.58 134.62 90)
+    (property "Value" "0.1uF" (at 195.58 134.62 90)
       (effects (font (size 1.27 1.27)))
     )
@@
       (effects (font (size 1.27 1.27)))
     )
-    (property "Value" "1uF" (at 195.58 121.92 90)
+    (property "Value" "0.1uF" (at 195.58 121.92 90)
       (effects (font (size 1.27 1.27)))
     )
@@
       (effects (font (size 1.27 1.27)))
     )
-    (property "Value" "1uF" (at 195.58 140.97 90)
-      (effects (font (size 1.27 1.27)))
-    )
+    (property "Value" "0.1uF" (at 195.58 140.97 90)
+      (effects (font (size 1.27 1.27)))
+    )
