File: appleii.vga/appleii.vga.kicad_sch (KiCad schematic)
At the start: 32 parts, among them J1 BUS_APPLE_II, J2 Conn_01x25, J3 Conn_01x25, J4 Conn_01x08, J5 Conn_01x03, Q1 DMG2305UX, U1 74LVC245A, U2 74LVC245A, U3 74LVC245A, U4 74LVC245A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

Commit message: update copyright in schematic
Other:
- company: swetland@frotz.net -> (none)
Changed lines of the file:
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@@
     (date "2023-07-13")
     (rev "v1.1.0")
-    (company "swetland@frotz.net")
+    (comment 1 "Licensed under the MIT-0 License")
+    (comment 2 "Copyright 2023, Brian Swetland <swetland@frotz.net>")
   )
   (junction (at 72.39 176.53) (diameter 0) (color 0 0 0 0)
